Commit message: Updated version

File: mar_description/urdf/mar_model.urdf (robot description, URDF)
Before this commit: robot MAR, 10 links, 9 joints
Joints:
- joint base_to_drive_compartment: origin xyz=0 0 -0.0025 -> xyz=0.03 0 -0.0025

File: mar_description/urdf/mar_model_sim.urdf (robot description, URDF)
Before this commit: robot MAR, 12 links, 11 joints
Joints:
- joint base_to_drive_compartment: origin xyz=0 0 -0.0025 -> xyz=0.03 0 -0.0025
